File: eagle/domotica/Master.sch (EAGLE design)
At the start: 1 part, among them IC1 MEGA8535-P

Commit message: modified master Branch to com_usb
Parts:
- added IC2, IC3, IC4, IC5, IC6, IC7, IC8, IC9: MEGA8535-P, librarie:MEGA8535-P
Connections:
- new net AREF: IC1.AREF, IC2.AREF, IC3.AREF, IC4.AREF, IC5.AREF, IC6.AREF, IC7.AREF, IC8.AREF, IC9.AREF
- new net AVCC: IC1.AVCC, IC2.AVCC, IC3.AVCC, IC4.AVCC, IC5.AVCC, IC6.AVCC, IC7.AVCC, IC8.AVCC, IC9.AVCC
- new net GND: IC1.GND, IC1.GND@1, IC2.GND, IC2.GND@1, IC3.GND, IC3.GND@1, IC4.GND, IC4.GND@1, IC5.GND, IC5.GND@1, IC6.GND, IC6.GND@1, IC7.GND, IC7.GND@1, IC8.GND, IC8.GND@1, IC9.GND, IC9.GND@1
- new net S0_0C0: IC2.(AIN0/OC0)PB2
- new net S0_0C1A: IC2.(OC1A)PD5
- new net S0_0C2: IC2.(OC2)PD7
- new net S0_PB0: IC2.(T0/XCK)PB0
- new net S0_PB1: IC2.(T1)PB1
- new net S0_PB3: IC2.(AIN1/INT2)PB3
- new net S0_PD0: IC2.(RXD)PD0
- new net S0_PD1: IC2.(TXD)PD1
- new net S0_PD2: IC2.(INT0)PD2
- new net S0_PD3: IC2.(INT1)PD3
- new net S0_PD4: IC2.(OC1B)PD4
- new net S0_PD6: IC2.(ICP)PD6
- new net SS0: IC1.(SCL)PC0, IC2.(SS)PB4
- new net SS1: IC1.(SDA)PC1, IC3.(SS)PB4
- new net SS2: IC1.PC2, IC4.(SS)PB4
- new net SS3: IC1.PC3, IC5.(SS)PB4
- new net SS4: IC1.PC4, IC6.(SS)PB4
- new net SS5: IC1.PC5, IC7.(SS)PB4
- new net SS6: IC1.(TOSC1)PC6, IC8.(SS)PB4
- new net SS7: IC1.(TOSC2)PC7, IC9.(SS)PB4
- new net USB_D+: IC1.(INT0)PD2
- new net USB_D-: IC1.(INT1)PD3
- new net VCC: IC1.VCC, IC2.VCC, IC3.VCC, IC4.VCC, IC5.VCC, IC6.VCC, IC7.VCC, IC8.VCC, IC9.VCC
- net MISO: now also IC2.(MISO)PB6, IC3.(MISO)PB6, IC4.(MISO)PB6, IC5.(MISO)PB6, IC6.(MISO)PB6, IC7.(MISO)PB6, IC8.(MISO)PB6, IC9.(MISO)PB6
- net MOSI: now also IC2.(MOSI)PB5, IC3.(MOSI)PB5, IC4.(MOSI)PB5, IC5.(MOSI)PB5, IC6.(MOSI)PB5, IC7.(MOSI)PB5, IC8.(MOSI)PB5, IC9.(MOSI)PB5
- net SCK: now also IC2.(SCK)PB7, IC3.(SCK)PB7, IC4.(SCK)PB7, IC5.(SCK)PB7, IC6.(SCK)PB7, IC7.(SCK)PB7, IC8.(SCK)PB7, IC9.(SCK)PB7
Other:
- note added: "Charlieplexing"
- note added: "PWM"
